Commit message: Some changes made to run restaurant simulation
Added urdf model instead of xacro, important changes are made in restaurant2.world to spawn robot succesfully and etc

File: urdf/bot.urdf.xacro (robot description, xacro)
@@ -1,4 +1,4 @@
 <?xml version='1.0'?>
-<robot name="waiter_bot" xmlns:xacro="http://www.ros.org/wiki/xacro">
+<robot name="bot" xmlns:xacro="http://www.ros.org/wiki/xacro">
 <xacro:property name="camera_link" value="0.01"/>
 <xacro:property name="camera_mass" value="0.1"/>
@@ -27,5 +27,5 @@
       <origin xyz="-0.205 -0.358 0" rpy="1.57 0 1.57"/>
       <geometry>
-        <mesh filename="package://dualwheelbot/meshes/marses_robot.stl" scale="0.001 0.001 0.001"/>
+        <mesh filename="package://waiter_bot/meshes/marses_robot.stl" scale="0.001 0.001 0.001"/>
       </geometry>
     </visual>
@@ -172,5 +172,5 @@
       <origin xyz="0 0 0" rpy="0 0 0"/>
       <geometry>
-        <mesh filename="package://dualwheelbot/meshes/hokuyo.dae"/>
+        <mesh filename="package://waiter_bot/meshes/hokuyo.dae"/>
       </geometry>
     </visual>
